File: RD53B_Quad_ZIF_to_ERF8_Data_Adapter.kicad_sch (KiCad schematic)
At the start: 15 parts, among them J2 Conn_02x01, J3 Conn_02x02_Odd_Even, J4 Conn_02x04_Odd_Even, J5 ERF8-050-01-X-D-EM2-TR, J6 Conn_02x01

Commit message: Remove biase resistors and change optoboard grounding
Parts:
- removed R1, R13, R14, R15, R16, R2, R7, R8: 10k, Resistor_SMD:R_0805_2012Metric, symbol Device:R

Commit message: Update
Parts:
- J_conn1: value ConnSingle -> Module ZIF connector
Changed lines of the file:
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@@
       (effects (font (size 1.524 1.524)))
     )
-    (property "Value" "ConnSingle" (id 1) (at 134.62 34.29 0)
+    (property "Value" "Module ZIF connector" (id 1) (at 134.62 34.29 0)
       (effects (font (size 1.524 1.524)))
     )
@@
     )
     (path "/1fd3e61b-118c-43f6-8a6f-bed7546351eb"
-      (reference "J_conn1") (unit 1) (value "ConnSingle") (footprint "Library:Molex-502598-3993")
-    )
-  )
+      (reference "J_conn1") (unit 1) (value "Module ZIF connector") (footprint "Library:Molex-502598-3993")
+    )
+  )
